File: schematic/shear_pcb.kicad_pcb (KiCad board)
At the start: 2 copper layers, 78.7 x 81.3 mm, 27 parts, among them J1 MOTOR1, J2 MOTOR2, J3 LCD_POWER, J4 VIN, J5 ENDSTOP1, J6 ENDSTOP2, J7 LCD_TOUCH, J8 LCD_SPI, U1 Teensy3.5, U2 AMIS30542, U3 AMIS30542, U4 R-785.0-1.0

Commit message: Add step file for CAD work
Parts:
- moved J4 5.08 mm to (179.7, 120.7), turned to 0 degrees
Routing:
- net VDC: track 178.5 -> 185.5 mm
Changed lines of the file:
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@@
     (thickness 1.6)
     (drawings 4)
-    (tracks 103)
+    (tracks 102)
     (zones 0)
     (modules 27)
@@
   )
   (module TerminalBlock:TerminalBlock_bornier-2_P5.08mm (layer F.Cu)
-    (at 184.785 120.65 180)
+    (at 179.705 120.65)
     (descr "simple 2-pin terminal block, pitch 5.08mm, revamped version of bornier2")
     (tags "terminal block bornier2")
@@
       (effects (font (size 1 1) (thickness 0.15)))
     )
-    (pad 2 thru_hole circle (at 5.08 0 180) (size 3 3) (drill 1.52) (layers *.Cu *.Mask)
+    (pad 2 thru_hole circle (at 5.08 0) (size 3 3) (drill 1.52) (layers *.Cu *.Mask)
       (net 22 VDC))
-    (pad 1 thru_hole rect (at 0 0 180) (size 3 3) (drill 1.52) (layers *.Cu *.Mask)
+    (pad 1 thru_hole rect (at 0 0) (size 3 3) (drill 1.52) (layers *.Cu *.Mask)
       (net 1 GND))
     (model ${KISYS3DMOD}/TerminalBlock.3dshapes/TerminalBlock_bornier-2_P5.08mm.wrl
@@
   (segment (start 150.62 59.18) (end 150.495 59.055) (width 1) (layer B.Cu) (net 22))
   (segment (start 150.62 63.5) (end 150.62 59.18) (width 1) (layer B.Cu) (net 22))
-  (segment (start 177.8 118.745) (end 179.705 120.65) (width 1) (layer B.Cu) (net 22))
-  (segment (start 161.925 121.285) (end 164.465 118.745) (width 1) (layer B.Cu) (net 22))
-  (segment (start 172.72 121.285) (end 175.26 118.745) (width 1) (layer B.Cu) (net 22))
-  (segment (start 164.465 118.745) (end 175.26 118.745) (width 1) (layer B.Cu) (net 22))
-  (segment (start 175.26 118.745) (end 177.8 118.745) (width 1) (layer B.Cu) (net 22))
   (segment (start 193.04 65.88) (end 193.04 61.755) (width 1) (layer F.Cu) (net 22))
   (segment (start 193.04 61.755) (end 183.99 52.705) (width 1) (layer F.Cu) (net 22))
   (segment (start 183.99 52.705) (end 182.245 52.705) (width 1) (layer F.Cu) (net 22))
-  (segment (start 193.04 92.235) (end 193.04 96.36) (width 1) (layer F.Cu) (net 22))
-  (segment (start 193.04 92.235) (end 184.15 83.345) (width 1) (layer F.Cu) (net 22))
-  (segment (start 182.405 83.345) (end 182.245 83.185) (width 1) (layer F.Cu) (net 22))
-  (segment (start 184.15 83.345) (end 182.405 83.345) (width 1) (layer F.Cu) (net 22))
-  (segment (start 179.705 109.695) (end 193.04 96.36) (width 1) (layer F.Cu) (net 22))
-  (segment (start 179.705 120.65) (end 179.705 109.695) (width 1) (layer F.Cu) (net 22))
-  (segment (start 184.15 74.77) (end 193.04 65.88) (width 1) (layer F.Cu) (net 22))
-  (segment (start 184.15 83.345) (end 184.15 74.77) (width 1) (layer F.Cu) (net 22))
   (segment (start 150.62 109.98) (end 161.925 121.285) (width 1) (layer B.Cu) (net 22))
   (segment (start 150.62 63.5) (end 150.62 109.98) (width 1) (layer B.Cu) (net 22))
+  (segment (start 183.99 83.185) (end 182.245 83.185) (width 1) (layer F.Cu) (net 22))
+  (segment (start 184.15 74.77) (end 193.04 65.88) (width 1) (layer F.Cu) (net 22))
+  (segment (start 193.04 92.235) (end 184.15 83.345) (width 1) (layer F.Cu) (net 22))
+  (segment (start 184.15 83.345) (end 184.15 74.77) (width 1) (layer F.Cu) (net 22))
+  (segment (start 193.04 96.36) (end 193.04 92.235) (width 1) (layer F.Cu) (net 22))
+  (segment (start 184.785 104.615) (end 193.04 96.36) (width 1) (layer F.Cu) (net 22))
+  (segment (start 184.785 120.65) (end 184.785 104.615) (width 1) (layer F.Cu) (net 22))
+  (segment (start 177.165 116.84) (end 172.72 121.285) (width 1) (layer B.Cu) (net 22))
+  (segment (start 161.925 121.285) (end 166.37 116.84) (width 1) (layer B.Cu) (net 22))
+  (segment (start 166.37 116.84) (end 177.165 116.84) (width 1) (layer B.Cu) (net 22))
+  (segment (start 180.975 116.84) (end 184.785 120.65) (width 1) (layer B.Cu) (net 22))
+  (segment (start 177.165 116.84) (end 180.975 116.84) (width 1) (layer B.Cu) (net 22))
   (segment (start 156.21 117.475) (end 144.78 106.045) (width 0.3) (layer F.Cu) (net 23))
   (segment (start 159.385 117.475) (end 156.21 117.475) (width 0.3) (layer F.Cu) (net 23))
