File: schematic/shear_pcb.kicad_pcb (KiCad board)
At the start: 2 copper layers, 78.7 x 81.3 mm, 27 parts, among them J1 MOTOR1, J2 MOTOR2, J3 LCD_POWER, J4 VIN, J5 ENDSTOP1, J6 ENDSTOP2, J7 LCD_TOUCH, J8 LCD_SPI, U1 Teensy3.5, U2 AMIS30542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

Commit message: Latest stable board and firmware
Parts:
- removed the J1 at (186.1, 67.9)
- removed the J2 at (186.1, 98.4)
- added G***: LOGO, CurieOS:CurieOS, F.Cu at (125.1, 81.3)
- added J7: FAN, Connector_JST:JST_EH_B2B-EH-A_1x02_P2.50mm_Vertical, F.Cu at (182.2, 110.5)
- moved C1 60.4 mm to (131.9, 106.0), turned to 180 degrees
- moved D1 55.3 mm to (132.3, 103.5), turned to 180 degrees
- moved J5 54.6 mm to (156.2, 55.9), turned to 180 degrees
- moved U4 51.0 mm to (127.6, 99.1), turned to 270 degrees
- moved C3 46.4 mm to (126.1, 95.2), turned to 180 degrees
- moved J4 42.3 mm to (156.2, 64.8), turned to 180 degrees
- moved C2 39.9 mm to (132.3, 95.2), turned to 0 degrees
- moved L1 35.7 mm to (129.2, 90.8), turned to 180 degrees
- moved J6 35.3 mm to (156.2, 81.3), turned to 180 degrees
- moved U2 30.7 mm to (174.6, 92.1)
- moved U3 30.7 mm to (174.6, 61.6)
- moved C7 10.2 mm to (192.4, 69.2), turned to 270 degrees
- moved C6 8.91 mm to (192.4, 59.7), turned to 90 degrees
- moved U1 7.62 mm to (144.8, 76.8), turned to 90 degrees
- moved J1 2.54 mm to (179.7, 118.1)
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- renumbered J4 to J1, J5 to J2, J6 to J3, J3 to J4, J7 to J5, J8 to J6
Connections:
- U1 pad 19: (no net) -> CLK
- U1 pad 2: (no net) -> END1
- U1 pad 3: (no net) -> END2
- U1 pad 30: END1 -> (no net)
- U1 pad 31: END2 -> (no net)
- U1 pad 40: CLK -> (no net)
- U1 pad 43: DIR2 -> (no net)
- U1 pad 44: STEP2 -> (no net)
- U1 pad 49: DIR1 -> (no net)
- U1 pad 5: (no net) -> DIR1
- U1 pad 50: STEP1 -> (no net)
- U1 pad 6: (no net) -> STEP1
- U1 pad 8: (no net) -> DIR2
- U1 pad 9: (no net) -> STEP2
- U2 pad 16: Net-(J1-Pad4) -> (no net)
- U2 pad 17: Net-(J1-Pad3) -> (no net)
- U2 pad 18: Net-(J1-Pad2) -> (no net)
- U2 pad 19: Net-(J1-Pad1) -> (no net)
- U3 pad 16: Net-(J2-Pad4) -> (no net)
- U3 pad 17: Net-(J2-Pad3) -> (no net)
- U3 pad 18: Net-(J2-Pad2) -> (no net)
- U3 pad 19: Net-(J2-Pad1) -> (no net)
Routing:
- net CLK: track 79.5 -> 48.1 mm, vias 1 -> 0
- net MISO: track 77.3 -> 57.8 mm
- net STEP2: track 19.9 -> 38.5 mm
- net DIR2: track 19.9 -> 38.2 mm
- net MOSI: track 77.4 -> 59.4 mm, vias 2 -> 1
- net CS3: track 16.7 -> 28.2 mm
- net END2: track 35.0 -> 27.4 mm
- net END1: track 23.1 -> 18.1 mm
- net CS2: track 26.4 -> 31.3 mm
- net XP: track 8.67 -> 4.60 mm
- net YM: track 8.67 -> 4.60 mm
- net Net-(J2-Pad4): track 3.81 -> 0.00 mm
- net Net-(J2-Pad3): track 3.81 -> 0.00 mm
- net Net-(J2-Pad2): track 3.81 -> 0.00 mm
- net Net-(J2-Pad1): track 3.81 -> 0.00 mm
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Other:
- net class Default: via_drill 0.25 -> 0.3
- net class Motor removed
- net class Power: clearance 0.2 -> 0.5; trace_width 1 -> 1.5; via_dia 1.2 -> 1.7; via_drill 0.8 -> 1
- board text added: "Shear Backstop Controller PCB V2"
